Commit message: MVP

File: rove_mvp_engine/data/robot.urdf (robot description, URDF)
Before this commit: robot rove_cursed_aaaah_goofy_design, 39 links, 38 joints
Joints:
- joint joint_revolute_10: origin xyz=-0.4 0.27 0.388 rpy=0 0 0 -> xyz=-0.4 0.27 0.388 rpy=3.14159 2.65359e-06 3.14159
- joint joint_revolute_11: origin xyz=-0.7 0.255 0.378 rpy=0 0 0 -> xyz=-0.7 0.255 0.378 rpy=3.14159 -2.65359e-06 3.14159
